Commit message: added getDeviceInfo for better localization

File: turtlebot_description/robots/kobuki_hexagons_kinect.urdf.xacro (robot description, xacro)
@@ -7,5 +7,5 @@
 <robot name="turtlebot" xmlns:xacro="http://ros.org/wiki/xacro">
   <xacro:include filename="$(find amr_x_communication)/turtlebot_description/urdf/turtlebot_common_library.urdf.xacro" />
-  <xacro:include filename="$(find amr_x_communication)/turtlebot_description/urdf/kobuki.urdf.xacro" />
+  <xacro:include filename="$(find amr_x_communication)/kobuki_description/urdf/kobuki.urdf.xacro" />
   <xacro:include filename="$(find amr_x_communication)/turtlebot_description/urdf/stacks/hexagons.urdf.xacro"/>
   <xacro:include filename="$(find amr_x_communication)/turtlebot_description/urdf/sensors/kinect.urdf.xacro"/>

File: turtlebot_description/urdf/sensors/hokuyo.urdf.xacro (robot description, xacro)
@@ -1,13 +1,13 @@
 <?xml version="1.0"?>
 <robot name="sensor_hokuyo" xmlns:xacro="http://ros.org/wiki/xacro">
-  <xacro:include filename="$(find amr_x_communication)/turtlebot_description/urdf/turtlebot_gazebo.urdf.xacro"/>
-  <xacro:include filename="$(find amr_x_communication)/turtlebot_description/urdf/turtlebot_properties.urdf.xacro"/>
-  <xacro:property name="hokuyo_cam_py" value="-0.0125"/>
-  <!-- Parameterised in part by the values in turtlebot_properties.urdf.xacro -->
-  <xacro:macro name="sensor_hokuyo" params="parent">
+<xacro:include filename="$(find amr_x_communication)/turtlebot_description/urdf/turtlebot_gazebo.urdf.xacro"/>
+<xacro:include filename="$(find amr_x_communication)/turtlebot_description/urdf/turtlebot_properties.urdf.xacro"/>
+<xacro:property name="hokuyo_cam_py" value="-0.0125"/>
+<!-- Parameterised in part by the values in turtlebot_properties.urdf.xacro -->
+<xacro:macro name="sensor_hokuyo" params="parent">
   <joint name="hokuyo_joint" type="fixed">
     <axis xyz="0 1 0" />
-    <origin xyz="0 0 ${height3 - axel_offset/2}" rpy="0 0 0"/>
-    <parent link="link3"/>
+    <origin xyz="0.1 0 0.22" rpy="0 0 0"/>
+    <parent link="base_link"/>
     <child link="hokuyo_link"/>
   </joint>
@@ -23,5 +23,5 @@
       <origin xyz="0 0 0" rpy="0 0 0"/>
       <geometry>
-        <mesh filename="package://rrbot_description/meshes/hokuyo.dae"/>
+        <mesh filename="package://amr_x_communication/turtlebot_description/meshes/sensors/hokuyo.dae"/>
       </geometry>
     </visual>
@@ -32,4 +32,39 @@
     </inertial>
   </link>
-  </xacro:macro>
+  <gazebo reference="hokuyo_link">
+    <sensor type="ray" name="head_hokuyo_sensor">
+      <pose>0 0 0 0 0 0</pose>
+      <visualize>true</visualize>
+      <update_rate>40</update_rate>
+      <ray>
+        <scan>
+          <horizontal>
+            <samples>90</samples>
+            <resolution>1</resolution>
+            <min_angle>-1.57079632679</min_angle>
+            <max_angle>1.57079632679</max_angle>
+          </horizontal>
+        </scan>
+        <range>
+          <min>0.40</min>
+          <max>5.0</max>
+          <resolution>0.01</resolution>
+        </range>
+        <noise>
+          <type>gaussian</type>
+          <!-- Noise parameters based on published spec for Hokuyo laser
+               achieving "+-30mm" accuracy at range < 10m.  A mean of 0.0m and
+               stddev of 0.01m will put 99.7% of samples within 0.03m of the true
+               reading. -->
+          <mean>0.0</mean>
+          <stddev>0.02</stddev>
+        </noise>
+      </ray>
+      <plugin name="gazebo_ros_head_hokuyo_controller" filename="libgazebo_ros_laser.so">
+        <topicName>scan</topicName>
+        <frameName>hokuyo_link</frameName>
+      </plugin>
+    </sensor>
+  </gazebo>
+</xacro:macro>
 </robot>
